File: Hardware/PCB/ST_KiCad/ST_KiCad.sch (KiCad schematic (older format))
At the start: 6 parts

Commit message: small update
Parts:
- C1, C2, C3: renamed from C?; footprint (none) -> Capacitor_THT:C_Radial_D12.5mm_H20.0mm_P5.00mm
- D1: renamed from D?; footprint (none) -> Diode_SMD:D_SMA
- L1: renamed from L?; footprint (none) -> Inductor_SMD:L_12x12mm_H8mm
- gave numbers to parts that had none: 1
Changed lines of the file:
@@
 $EndDescr
 $Comp
-L Regulator_Switching:LM2596S-5 U?
+L Regulator_Switching:LM2596S-5 U1
 U 1 1 6058F530
 P 3100 1650
-F 0 "U?" H 3100 2017 50  0000 C CNN
+F 0 "U1" H 3100 2017 50  0000 C CNN
 F 1 "LM2596S-5" H 3100 1926 50  0000 C CNN
 F 2 "Package_TO_SOT_SMD:TO-263-5_TabPin3" H 3150 1400 50  0001 L CIN
@@
 	2600 1550 2050 1550
 $Comp
-L Device:D_Schottky D?
+L Device:D_Schottky D1
 U 1 1 605930F8
 P 3750 1950
-F 0 "D?" V 3704 2030 50  0000 L CNN
+F 0 "D1" V 3704 2030 50  0000 L CNN
 F 1 "D_Schottky" V 3795 2030 50  0000 L CNN
-F 2 "" H 3750 1950 50  0001 C CNN
+F 2 "Diode_SMD:D_SMA" H 3750 1950 50  0001 C CNN
 F 3 "~" H 3750 1950 50  0001 C CNN
 	1    3750 1950
@@
 $EndComp
 $Comp
-L pspice:INDUCTOR L?
+L pspice:INDUCTOR L1
 U 1 1 60594D64
 P 4150 1750
-F 0 "L?" H 4150 1965 50  0000 C CNN
+F 0 "L1" H 4150 1965 50  0000 C CNN
 F 1 "33u" H 4150 1874 50  0000 C CNN
-F 2 "" H 4150 1750 50  0001 C CNN
+F 2 "Inductor_SMD:L_12x12mm_H8mm" H 4150 1750 50  0001 C CNN
 F 3 "~" H 4150 1750 50  0001 C CNN
 	1    4150 1750
@@
 	3750 2100 3750 2300
 $Comp
-L power:GND #PWR?
+L power:GND #PWR06
 U 1 1 6059638C
 P 3750 2300
-F 0 "#PWR?" H 3750 2050 50  0001 C CNN
+F 0 "#PWR06" H 3750 2050 50  0001 C CNN
 F 1 "GND" H 3755 2127 50  0000 C CNN
 F 2 "" H 3750 2300 50  0001 C CNN
@@
 $EndComp
 $Comp
-L power:GND #PWR?
+L power:GND #PWR05
 U 1 1 60596A8F
 P 3100 2300
-F 0 "#PWR?" H 3100 2050 50  0001 C CNN
+F 0 "#PWR05" H 3100 2050 50  0001 C CNN
 F 1 "GND" H 3105 2127 50  0000 C CNN
 F 2 "" H 3100 2300 50  0001 C CNN
@@
 $EndComp
 $Comp
-L power:GND #PWR?
+L power:GND #PWR04
 U 1 1 60596F9D
 P 2450 2300
-F 0 "#PWR?" H 2450 2050 50  0001 C CNN
+F 0 "#PWR04" H 2450 2050 50  0001 C CNN
 F 1 "GND" H 2455 2127 50  0000 C CNN
 F 2 "" H 2450 2300 50  0001 C CNN
@@
 $EndComp
 $Comp
-L Device:C C?
+L Device:C C3
 U 1 1 60598E9E
 P 4600 1950
-F 0 "C?" H 4715 1996 50  0000 L CNN
+F 0 "C3" H 4715 1996 50  0000 L CNN
 F 1 "330u" H 4715 1905 50  0000 L CNN
-F 2 "" H 4638 1800 50  0001 C CNN
+F 2 "Capacitor_THT:C_Radial_D12.5mm_H20.0mm_P5.00mm" H 4638 1800 50  0001 C CNN
 F 3 "~" H 4600 1950 50  0001 C CNN
 	1    4600 1950
@@
 $EndComp
 $Comp
-L Device:C C?
+L Device:C C2
 U 1 1 60599319
 P 2050 1950
-F 0 "C?" H 2165 1996 50  0000 L CNN
+F 0 "C2" H 2165 1996 50  0000 L CNN
 F 1 "330u" H 2165 1905 50  0000 L CNN
-F 2 "" H 2088 1800 50  0001 C CNN
+F 2 "Capacitor_THT:C_Radial_D12.5mm_H20.0mm_P5.00mm" H 2088 1800 50  0001 C CNN
 F 3 "~" H 2050 1950 50  0001 C CNN
 	1    2050 1950
@@
 	4600 2100 4600 2300
 $Comp
-L power:GND #PWR?
+L power:GND #PWR07
 U 1 1 6059AB5A
 P 4600 2300
-F 0 "#PWR?" H 4600 2050 50  0001 C CNN
+F 0 "#PWR07" H 4600 2050 50  0001 C CNN
 F 1 "GND" H 4605 2127 50  0000 C CNN
 F 2 "" H 4600 2300 50  0001 C CNN
@@
 	2050 2100 2050 2300
 $Comp
-L power:GND #PWR?
+L power:GND #PWR03
 U 1 1 6059B05B
 P 2050 2300
-F 0 "#PWR?" H 2050 2050 50  0001 C CNN
+F 0 "#PWR03" H 2050 2050 50  0001 C CNN
 F 1 "GND" H 2055 2127 50  0000 C CNN
 F 2 "" H 2050 2300 50  0001 C CNN
@@
 Connection ~ 2050 1550
 $Comp
-L Device:C C?
+L Device:C C1
 U 1 1 6059EE3E
 P 1750 1950
-F 0 "C?" H 1550 2000 50  0000 L CNN
+F 0 "C1" H 1550 2000 50  0000 L CNN
 F 1 "330u" H 1450 1900 50  0000 L CNN
-F 2 "" H 1788 1800 50  0001 C CNN
+F 2 "Capacitor_THT:C_Radial_D12.5mm_H20.0mm_P5.00mm" H 1788 1800 50  0001 C CNN
 F 3 "~" H 1750 1950 50  0001 C CNN
 	1    1750 1950
@@
 	1750 2100 1750 2300
 $Comp
-L power:GND #PWR?
+L power:GND #PWR02
 U 1 1 6059F8E9
 P 1750 2300
-F 0 "#PWR?" H 1750 2050 50  0001 C CNN
+F 0 "#PWR02" H 1750 2050 50  0001 C CNN
 F 1 "GND" H 1755 2127 50  0000 C CNN
 F 2 "" H 1750 2300 50  0001 C CNN
@@
 $EndComp
 $Comp
-L power:+5V #PWR?
+L power:+5V #PWR08
 U 1 1 605A9B12
 P 5050 1200
-F 0 "#PWR?" H 5050 1050 50  0001 C CNN
+F 0 "#PWR08" H 5050 1050 50  0001 C CNN
 F 1 "+5V" H 5065 1373 50  0000 C CNN
 F 2 "" H 5050 1200 50  0001 C CNN
@@
 	5050 1200 5050 1750
 $Comp
-L power:+12V #PWR?
+L power:+12V #PWR01
 U 1 1 605AB153
 P 1350 1200
-F 0 "#PWR?" H 1350 1050 50  0001 C CNN
+F 0 "#PWR01" H 1350 1050 50  0001 C CNN
 F 1 "+12V" H 1365 1373 50  0000 C CNN
 F 2 "" H 1350 1200 50  0001 C CNN

Commit message: teriyaki init
Parts:
- added A1, A2: Pololu_Breakout_DRV8825, Module:Pololu_Breakout-16_15.2x20.3mm, symbol Driver_Motor:Pololu_Breakout_DRV8825
- added C?: C_Small, symbol Device:C_Small
- added D?: D_Schottky_Small, symbol Device:D_Schottky_Small
- added F?: Polyfuse_Small, symbol Device:Polyfuse_Small
- added J?: POWER_JACK, POWER_JACK_PTH, symbol SparkFun-Connectors:POWER_JACK
- added J?: USB_B_Micro, symbol Connector:USB_B_Micro
- added J?: USB_A, symbol Connector:USB_A
- added LED_DRV_ELV1, LED_RED_12V1, LED_RED_3V3?, LED_RED_5V1, LED_RED_5V?: LED, LED_SMD:LED_0805_2012Metric, symbol Device:LED
- added Q?: AO3401A, Package_TO_SOT_SMD:SOT-23, symbol Transistor_FET:AO3401A
- added R1, R2, R? (x2): 1k, symbol Device:R
- added R3: R, symbol Device:R
- added TP? (x6): TestPoint, symbol Connector:TestPoint
- added U2: STM8L051F3P6, Package_SO:TSSOP-20_4.4x6.5mm_P0.65mm, symbol MCU_ST_STM8:STM8L051F3P
- added U?: FT232RL, Package_SO:SSOP-28_5.3x10.2mm_P0.65mm, symbol Interface_USB:FT232RL
Connections:
- net labels added: +3.3V, +3V3, +5P, STM8_RX, STM8_TX, USB_D+, USB_D-
- wire segments 22 -> 77
- no-connect marks 0 -> 19
Other:
- note added: "12V --> 5V, 3A SMPS"
- note added: "12V Connector"
- note added: "For external connector"
- note added: "Power LEDs"
- note added: "STM8 Supply"
- note added: "USB A Out"
- note added: "and supply test points"
- note added: "micro USB IN"
- moved on the sheet: C1, C2, C3, D1, L1, U1
