File: Hardware/PCB/Teriyaki_prototype/teriyaki.kicad_pcb (KiCad board)
At the start: 4 copper layers, 60 x 45 mm, 56 parts, among them J1 USB_B_Micro, J2 Conn_01x02, J3 Conn_01x10, J4 Conn_01x02, U1 XL1509, U2 STM8S105K6, U3 FT232RL, U4 USBLC6-2SC6, Y1 16MHz

Commit message: update
Parts:
- moved J2 24.7 mm to (121.7, 103.0), turned to 0 degrees
- moved LED_3V31 16.6 mm to (114.3, 112.1)
- moved R16 16.6 mm to (114.2, 110.0)
- moved R3 12.7 mm to (125.3, 103.0)
- moved R4 12.5 mm to (125.3, 105.6)
- moved C7 11.9 mm to (114.3, 116.8), turned to 270 degrees
- moved LED_RX1 6.72 mm to (112.6, 99.9)
- moved LED_TX1 6.72 mm to (112.6, 97.5)
- moved R5 6.72 mm to (116.1, 97.5)
- moved R6 6.72 mm to (116.1, 99.9)
- moved LED1 3.45 mm to (112.6, 106.4)
- moved LED2 3.45 mm to (112.6, 104.4)
- moved LED3 3.45 mm to (112.6, 102.2)
- moved R11 3.45 mm to (116.1, 104.4)
- moved R13 3.45 mm to (116.1, 102.2)
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Routing:
- net STM8_RX: track 35.6 -> 8.49 mm, vias 2 -> 1
- net STM8_TX: track 32.9 -> 18.4 mm, vias 2 -> 1
- net Net-(R4-Pad2): track 18.4 -> 5.92 mm
- net Net-(R3-Pad2): track 14.1 -> 2.76 mm
- net +3V3: track 74.8 -> 67.0 mm
- net CBUS1: track 8.72 -> 15.8 mm
- net CBUS0: track 7.33 -> 14.1 mm
- net GPIO_B2: track 29.8 -> 33.4 mm
- net GPIO_B1: track 25.0 -> 28.7 mm
- net GPIO_B0: track 20.0 -> 22.5 mm
