File: Hardware/PCB/Teriyaki_prototype/teriyaki.sch (KiCad schematic (older format))
At the start: 55 parts, among them J1 USB_B_Micro, J2 Conn_01x02, J3 Conn_01x10, J4 Conn_01x02, U1 XL1509, U2 STM8S105K6, U3 FT232RL, U4 USBLC6-2SC6, Y1 16MHz

Commit message: just a backup
Parts:
- U2: LCSC Part (none) -> C8254
Changed lines of the file:
@@
 F 2 "Package_QFP:LQFP-32_7x7mm_P0.8mm" H 8550 6050 50  0001 C CNN
 F 3 "" H 10550 3700 50  0001 C CNN
+F 4 "C8254" H 8500 4700 50  0001 C CNN "LCSC Part"
 	1    8500 4700
 	1    0    0    -1
