File: Hardware/PCB/Teriyaki_prototype_STM8_outOfStock_oof/teriyaki.sch (KiCad schematic (older format))
At the start: 55 parts, among them J1 USB_B_Micro, J2 Conn_01x02, J3 Conn_01x10, J4 Conn_01x02, U1 XL1509, U2 STM8S105K6, U3 FT232RL, U4 USBLC6-2SC6, Y1 16MHz

Commit message: created prototype board
Parts:
- removed C13: 1u, Capacitor_SMD:C_0603_1608Metric, symbol Device:C_Small
- removed U2: STM8S105K6, Package_QFP:LQFP-32_7x7mm_P0.8mm, symbol richiegreen:STM8S105K6
- added U2: STM8L051F3P6, Package_SO:TSSOP-20_4.4x6.5mm_P0.65mm, symbol MCU_ST_STM8:STM8L051F3P
Connections:
- net labels added: GPIO_PB3, GPIO_PB4, GPIO_PB5, GPIO_PB6, GPIO_PB7, GPIO_PC4, TIM2_CH1, TIM2_CH2, TIM3_CH1, TIM3_CH2
- net labels removed: GPIO_B0, GPIO_B1, GPIO_B2, GPIO_C1, GPIO_C2, GPIO_C3, GPIO_C4, GPIO_C5, GPIO_C6, GPIO_C7
- wire segments 160 -> 148
Other:
- moved on the sheet: C11, C12, R14, R15
